Commit message: feat: 图书馆机器人 GUI 地图点击 + 语音找书闭环
地图锚点与导航目标
* scripts/obstacle_anchor.py —— 从 maps/room.pgm 提取 4 个内部障碍物(桌椅/书架)
  锚点 + 净空足够且在主连通区内的停靠点,落 maps/bookmarks.json
* scripts/anchors_verify.py —— 邻域栅格可视化校验
* scripts/plan_check.py —— 直接复用导航栈 AStar8 验证停靠点 12 起点全可达

板端协议
* goal_bridge_node —— 新增任意坐标 goto 命令(map 系),同时保留旧的
  find_book+location(A/B/C/D)兼容;坐标超地图范围拒绝;地图边界从
  maps/room.yaml 静态读,/map 实时话题来一次更准一次
* robot_comm.send_goto_xy —— GUI 端派单新接口,旧 send_go_to 保留兼容

GUI
* map_view.py —— 新地图视图(PySide6 QGraphicsView 渲染 PGM),
  4 个书位彩色圆点 + 书名标注,点击任意点 → 像素 → map 坐标 → 派单
* GUI.py —— '🗺️ 地图' 按钮打开 MapViewWindow,'🔍 寻找图书' 按钮弹输入框,
  BookDetailPage '寻找图书' 优先用 bookmarks 坐标派单(无则用旧区号)

语音找书
* book_chat.py —— search 分支命中后顺手派单;意图补漏(我要找/请找/
  带我去/想看等);关键词清理
* book_ai.py —— search_books 返回 (reply, first_book_name),供派单取书名

未追踪文件保持不动(scripts/*.py 早期遗留、maps/*.pgm 太大不入库、
start_map.sh.bak、config/robot_lite.rviz 等)

File: src/robot_description/urdf/library_robot.urdf (robot description, URDF)
Before this commit: robot library_robot, 3 links, 2 joints
Joints:
- joint base_link_to_laser: origin xyz=0 0 0.25 rpy=0 0 0 -> xyz=0 0 0.25 rpy=0 0 3.14159265

Commit message: fix: 雷达朝向实测确认 + 编码器/膨胀半径/launch 修正
- URDF: 雷达朝向实测 theta_front≈155° -> yaw≈180° 正确, 注释由待确认改为已验证; inflation 统一为单一来源 0.28
- robot_nav_all.launch.py: enable_slam 重复声明合并; static_map_nav.launch.py 补 nav2_lifecycle_manager(原先 /map 永不发布)
- stm32_bridge: 新增 IMU(TYPE 0x04) 解析与 /imu/data 发布, 修 TYPE_ACK 撞号
- library_gui: TTS 播放设备按声卡名绑定(卡号会漂), 语音/地图模块更新
- scripts: 新增 encoder_calib.py(编码器标定+轮向符号验证)、lidar_yaw_check.py(雷达朝向判定)

File: src/robot_description/urdf/library_robot.urdf (robot description, URDF)
Before this commit: robot library_robot, 3 links, 2 joints
Links:
- link base_link: geometry collision box size=0.33 0.25 0.37; visual box size=0.33 0.25 0.37
Joints:
- joint base_link_to_laser: origin xyz=0 0 0.25 rpy=0 0 3.14159265 -> xyz=0 0 0.12 rpy=0 0 3.14159265
